File: counting-registers/schematics/flags-register/flags-register.sch (KiCad schematic (older format))
At the start: 13 parts

Commit message: updated documentation
Parts:
- gave numbers to parts that had none: 5
Changed lines of the file:
@@
 $EndDescr
 $Comp
-L 74xx:74LS173 U?
+L 74xx:74LS173 U5
 U 1 1 5FF57380
 P 5000 2825
-F 0 "U?" H 5225 3725 50  0000 C CNN
+F 0 "U5" H 5225 3725 50  0000 C CNN
 F 1 "74LS173" H 5225 3625 50  0000 C CNN
 F 2 "" H 5000 2825 50  0001 C CNN
@@
 Jf
 $Comp
-L 74xx:74LS08 U?
+L 74xx:74LS08 U1
 U 1 1 5FF59424
 P 775 2175
-F 0 "U?" H 775 2500 50  0000 C CNN
+F 0 "U1" H 775 2500 50  0000 C CNN
 F 1 "74LS08" H 775 2409 50  0000 C CNN
 F 2 "" H 775 2175 50  0001 C CNN
@@
 $EndComp
 $Comp
-L 74xx:74LS08 U?
+L 74xx:74LS08 U1
 U 2 1 5FF67906
 P 2175 2825
-F 0 "U?" H 2175 3150 50  0000 C CNN
+F 0 "U1" H 2175 3150 50  0000 C CNN
 F 1 "74LS08" H 2175 3059 50  0000 C CNN
 F 2 "" H 2175 2825 50  0001 C CNN
@@
 $EndComp
 $Comp
-L 74xx:74LS08 U?
+L 74xx:74LS08 U1
 U 3 1 5FF6A4A2
 P 2175 3375
-F 0 "U?" H 2175 3700 50  0000 C CNN
+F 0 "U1" H 2175 3700 50  0000 C CNN
 F 1 "74LS08" H 2175 3609 50  0000 C CNN
 F 2 "" H 2175 3375 50  0001 C CNN
@@
 	1500 3475 1875 3475
 $Comp
-L 4xxx:4075 U?
+L 4xxx:4075 U3
 U 1 1 5FF71A70
 P 2200 1575
-F 0 "U?" H 2375 1850 50  0000 C CNN
+F 0 "U3" H 2375 1850 50  0000 C CNN
 F 1 "74HCT4075" H 2500 1750 50  0000 C CNN
 F 2 "" H 2200 1575 50  0001 C CNN
@@
 	4425 3075 4425 3125
 $Comp
-L 4xxx:4075 U?
+L 4xxx:4075 U3
 U 2 1 5FF818FA
 P 2975 2825
-F 0 "U?" H 2975 3150 50  0000 C CNN
+F 0 "U3" H 2975 3150 50  0000 C CNN
 F 1 "74HCT4075" H 3100 3050 50  0000 C CNN
 F 2 "" H 2975 2825 50  0001 C CNN
@@
 	4325 1575 4325 3075
 $Comp
-L power:GND #PWR?
+L power:GND #PWR01
 U 1 1 5FF8B765
 P 4425 2825
-F 0 "#PWR?" H 4425 2575 50  0001 C CNN
+F 0 "#PWR01" H 4425 2575 50  0001 C CNN
 F 1 "GND" H 4525 2725 50  0000 C CNN
 F 2 "" H 4425 2825 50  0001 C CNN
@@
 Connection ~ 4425 2525
 $Comp
-L 74xx:74LS08 U?
+L 74xx:74LS08 U2
 U 1 1 5FF8E424
 P 850 3725
-F 0 "U?" H 850 4050 50  0000 C CNN
+F 0 "U2" H 850 4050 50  0000 C CNN
 F 1 "74LS08" H 850 3959 50  0000 C CNN
 F 2 "" H 850 3725 50  0001 C CNN
@@
 $EndComp
 $Comp
-L 74xx:74LS08 U?
+L 74xx:74LS08 U2
 U 2 1 5FF917B8
 P 2175 4475
-F 0 "U?" H 2175 4800 50  0000 C CNN
+F 0 "U2" H 2175 4800 50  0000 C CNN
 F 1 "74LS08" H 2175 4709 50  0000 C CNN
 F 2 "" H 2175 4475 50  0001 C CNN
@@
 $EndComp
 $Comp
-L 74xx:74LS08 U?
+L 74xx:74LS08 U2
 U 3 1 5FF936B4
 P 2175 5025
-F 0 "U?" H 2175 5350 50  0000 C CNN
+F 0 "U2" H 2175 5350 50  0000 C CNN
 F 1 "74LS08" H 2175 5259 50  0000 C CNN
 F 2 "" H 2175 5025 50  0001 C CNN
@@
 Connection ~ 1775 1675
 $Comp
-L 4xxx:4075 U?
+L 4xxx:4075 U3
 U 3 1 5FFB775B
 P 2975 4475
-F 0 "U?" H 2975 4800 50  0000 C CNN
+F 0 "U3" H 2975 4800 50  0000 C CNN
 F 1 "74HCT4075" H 3100 4700 50  0000 C CNN
 F 2 "" H 2975 4475 50  0001 C CNN
@@
 	5500 2325 5750 2325
 $Comp
-L power:VCC #PWR?
+L power:VCC #PWR02
 U 1 1 5FFCED59
 P 5000 1850
-F 0 "#PWR?" H 5000 1700 50  0001 C CNN
+F 0 "#PWR02" H 5000 1700 50  0001 C CNN
 F 1 "VCC" H 5015 2023 50  0000 C CNN
 F 2 "" H 5000 1850 50  0001 C CNN
@@
 $EndComp
 $Comp
-L power:GND #PWR?
+L power:GND #PWR03
 U 1 1 5FFCF87A
 P 5000 3800
-F 0 "#PWR?" H 5000 3550 50  0001 C CNN
+F 0 "#PWR03" H 5000 3550 50  0001 C CNN
 F 1 "GND" H 5005 3627 50  0000 C CNN
 F 2 "" H 5000 3800 50  0001 C CNN
@@
 NoConn ~ 5500 2525
 $Comp
-L 74xx:74LS08 U?
+L 74xx:74LS08 U1
 U 4 1 5FF2F669
 P 2175 2275
-F 0 "U?" H 2175 2600 50  0000 C CNN
+F 0 "U1" H 2175 2600 50  0000 C CNN
 F 1 "74LS08" H 2175 2509 50  0000 C CNN
 F 2 "" H 2175 2275 50  0001 C CNN
@@
 $EndComp
 $Comp
-L 74xx:74LS08 U?
+L 74xx:74LS08 U2
 U 4 1 5FF3CFCF
 P 2175 3925
-F 0 "U?" H 2175 4250 50  0000 C CNN
+F 0 "U2" H 2175 4250 50  0000 C CNN
 F 1 "74LS08" H 2175 4159 50  0000 C CNN
 F 2 "" H 2175 3925 50  0001 C CNN
@@
 $EndComp
 $Comp
-L 74xx:74LS04 U?
+L 74xx:74LS04 U4
 U 6 1 5FF445A8
 P 3200 1575
-F 0 "U?" H 3200 1892 50  0000 C CNN
+F 0 "U4" H 3200 1892 50  0000 C CNN
 F 1 "74LS04" H 3200 1801 50  0000 C CNN
 F 2 "" H 3200 1575 50  0001 C CNN
