File: ram-rom-upgrade/schematics/run-mode-selector-16bit/run-mode-selector-16bit.sch (KiCad schematic (older format))
At the start: 18 parts

Commit message: update ram-rom module documentation
Parts:
- gave numbers to parts that had none: 18
Changed lines of the file:
@@
 A15
 $Comp
-L 74xx:74LS157 U?
+L 74xx:74LS157 U1
 U 1 1 60588DDC
 P 2450 5200
-F 0 "U?" V 2825 4400 50  0000 L CNN
+F 0 "U1" V 2825 4400 50  0000 L CNN
 F 1 "74LS157" V 2450 5025 50  0000 L CNN
 F 2 "" H 2450 5200 50  0001 C CNN
@@
 $EndComp
 $Comp
-L 74xx:74LS157 U?
+L 74xx:74LS157 U2
 U 1 1 6058F2C6
 P 4625 5200
-F 0 "U?" V 5000 4400 50  0000 L CNN
+F 0 "U2" V 5000 4400 50  0000 L CNN
 F 1 "74LS157" V 4625 5025 50  0000 L CNN
 F 2 "" H 4625 5200 50  0001 C CNN
@@
 $EndComp
 $Comp
-L 74xx:74LS157 U?
+L 74xx:74LS157 U3
 U 1 1 60590082
 P 6725 5200
-F 0 "U?" V 7100 4400 50  0000 L CNN
+F 0 "U3" V 7100 4400 50  0000 L CNN
 F 1 "74LS157" V 6725 5025 50  0000 L CNN
 F 2 "" H 6725 5200 50  0001 C CNN
@@
 $EndComp
 $Comp
-L 74xx:74LS157 U?
+L 74xx:74LS157 U4
 U 1 1 60590658
 P 8775 5200
-F 0 "U?" V 9150 4400 50  0000 L CNN
+F 0 "U4" V 9150 4400 50  0000 L CNN
 F 1 "74LS157" V 8775 5025 50  0000 L CNN
 F 2 "" H 8775 5200 50  0001 C CNN
@@
 $EndComp
 $Comp
-L Switch:SW_DIP_x08 SW?
+L Switch:SW_DIP_x08 SW1
 U 1 1 60598F76
 P 950 3200
-F 0 "SW?" H 950 3867 50  0000 C CNN
+F 0 "SW1" H 950 3867 50  0000 C CNN
 F 1 "SW_DIP_x08" H 950 3776 50  0000 C CNN
 F 2 "" H 950 3200 50  0001 C CNN
@@
 $EndComp
 $Comp
-L Switch:SW_DIP_x08 SW?
+L Switch:SW_DIP_x08 SW2
 U 1 1 6059B235
 P 950 4150
-F 0 "SW?" H 950 3575 50  0000 C CNN
+F 0 "SW2" H 950 3575 50  0000 C CNN
 F 1 "SW_DIP_x08" H 950 3675 50  0000 C CNN
 F 2 "" H 950 4150 50  0001 C CNN
@@
 Connection ~ 650  4350
 $Comp
-L power:GND #PWR?
+L power:GND #PWR01
 U 1 1 60656D6C
 P 650 4800
-F 0 "#PWR?" H 650 4550 50  0001 C CNN
+F 0 "#PWR01" H 650 4550 50  0001 C CNN
 F 1 "GND" H 655 4627 50  0000 C CNN
 F 2 "" H 650 4800 50  0001 C CNN
@@
 	9375 6325 9375 5700
 $Comp
-L power:GND #PWR?
+L power:GND #PWR02
 U 1 1 606EC1D2
 P 1450 5200
-F 0 "#PWR?" H 1450 4950 50  0001 C CNN
+F 0 "#PWR02" H 1450 4950 50  0001 C CNN
 F 1 "GND" H 1455 5027 50  0000 C CNN
 F 2 "" H 1450 5200 50  0001 C CNN
@@
 Connection ~ 1450 5200
 $Comp
-L power:GND #PWR?
+L power:GND #PWR04
 U 1 1 606EC5FB
 P 3625 5200
-F 0 "#PWR?" H 3625 4950 50  0001 C CNN
+F 0 "#PWR04" H 3625 4950 50  0001 C CNN
 F 1 "GND" H 3630 5027 50  0000 C CNN
 F 2 "" H 3625 5200 50  0001 C CNN
@@
 Connection ~ 3625 5200
 $Comp
-L power:GND #PWR?
+L power:GND #PWR08
 U 1 1 606ECA30
 P 5725 5200
-F 0 "#PWR?" H 5725 4950 50  0001 C CNN
+F 0 "#PWR08" H 5725 4950 50  0001 C CNN
 F 1 "GND" H 5730 5027 50  0000 C CNN
 F 2 "" H 5725 5200 50  0001 C CNN
@@
 Connection ~ 5725 5200
 $Comp
-L power:GND #PWR?
+L power:GND #PWR011
 U 1 1 606ECE71
 P 7775 5200
-F 0 "#PWR?" H 7775 4950 50  0001 C CNN
+F 0 "#PWR011" H 7775 4950 50  0001 C CNN
 F 1 "GND" H 7780 5027 50  0000 C CNN
 F 2 "" H 7775 5200 50  0001 C CNN
@@
 PROG
 $Comp
-L power:VCC #PWR?
+L power:VCC #PWR012
 U 1 1 606F7246
 P 9675 5200
-F 0 "#PWR?" H 9675 5050 50  0001 C CNN
+F 0 "#PWR012" H 9675 5050 50  0001 C CNN
 F 1 "VCC" H 9690 5373 50  0000 C CNN
 F 2 "" H 9675 5200 50  0001 C CNN
@@
 $EndComp
 $Comp
-L power:VCC #PWR?
+L power:VCC #PWR010
 U 1 1 6072F5DD
 P 7625 5200
-F 0 "#PWR?" H 7625 5050 50  0001 C CNN
+F 0 "#PWR010" H 7625 5050 50  0001 C CNN
 F 1 "VCC" H 7640 5373 50  0000 C CNN
 F 2 "" H 7625 5200 50  0001 C CNN
@@
 $EndComp
 $Comp
-L power:VCC #PWR?
+L power:VCC #PWR07
 U 1 1 6072FAB1
 P 5525 5200
-F 0 "#PWR?" H 5525 5050 50  0001 C CNN
+F 0 "#PWR07" H 5525 5050 50  0001 C CNN
 F 1 "VCC" H 5540 5373 50  0000 C CNN
 F 2 "" H 5525 5200 50  0001 C CNN
@@
 $EndComp
 $Comp
-L power:VCC #PWR?
+L power:VCC #PWR03
 U 1 1 6072FF6A
 P 3350 5200
-F 0 "#PWR?" H 3350 5050 50  0001 C CNN
+F 0 "#PWR03" H 3350 5050 50  0001 C CNN
 F 1 "VCC" H 3365 5373 50  0000 C CNN
 F 2 "" H 3350 5200 50  0001 C CNN
@@
 	10925 4975 11050 4975
 $Comp
-L power:GND #PWR?
+L power:GND #PWR014
 U 1 1 60610629
 P 11050 4975
-F 0 "#PWR?" H 11050 4725 50  0001 C CNN
+F 0 "#PWR014" H 11050 4725 50  0001 C CNN
 F 1 "GND" H 11055 4802 50  0000 C CNN
 F 2 "" H 11050 4975 50  0001 C CNN
@@
 	10100 6075 10100 5975
 $Comp
-L power:VCC #PWR?
+L power:VCC #PWR013
 U 1 1 605F5E31
 P 10100 6075
-F 0 "#PWR?" H 10100 5925 50  0001 C CNN
+F 0 "#PWR013" H 10100 5925 50  0001 C CNN
 F 1 "VCC" H 10115 6248 50  0000 C CNN
 F 2 "" H 10100 6075 50  0001 C CNN
@@
 $EndComp
 $Comp
-L Device:R R?
+L Device:R R1
 U 1 1 605F5563
 P 9850 5700
-F 0 "R?" V 9750 5650 50  0000 L CNN
+F 0 "R1" V 9750 5650 50  0000 L CNN
 F 1 "1K" V 9850 5650 50  0000 L CNN
 F 2 "" V 9780 5700 50  0001 C CNN
@@
 $EndComp
 $Comp
-L Device:R R?
+L Device:R R2
 U 1 1 605F4E75
 P 10100 5700
-F 0 "R?" V 10000 5650 50  0000 L CNN
+F 0 "R2" V 10000 5650 50  0000 L CNN
 F 1 "220" V 10100 5625 50  0000 L CNN
 F 2 "" V 10030 5700 50  0001 C CNN
@@
 $EndComp
 $Comp
-L Device:R R?
+L Device:R R3
 U 1 1 605F477A
 P 10425 5700
-F 0 "R?" V 10325 5650 50  0000 L CNN
+F 0 "R3" V 10325 5650 50  0000 L CNN
 F 1 "220" V 10425 5625 50  0000 L CNN
 F 2 "" V 10355 5700 50  0001 C CNN
@@
 $EndComp
 $Comp
-L Device:LED_Small_ALT D?
+L Device:LED_Small_ALT D1
 U 1 1 605F3ADE
 P 10100 5375
-F 0 "D?" H 10150 5500 50  0000 R CNN
+F 0 "D1" H 10150 5500 50  0000 R CNN
 F 1 "RED" H 10225 5275 50  0000 R CNN
 F 2 "" V 10100 5375 50  0001 C CNN
@@
 $EndComp
 $Comp
-L Device:LED_Small_ALT D?
+L Device:LED_Small_ALT D2
 U 1 1 605F2267
 P 10425 5375
-F 0 "D?" H 10475 5500 50  0000 R CNN
+F 0 "D2" H 10475 5500 50  0000 R CNN
 F 1 "GREEN" H 10550 5275 50  0000 R CNN
 F 2 "" V 10425 5375 50  0001 C CNN
@@
 $EndComp
 $Comp
-L Switch:SW_SPDT SW?
+L Switch:SW_SPDT SW3
 U 1 1 605E7856
 P 10725 4975
-F 0 "SW?" H 10725 5260 50  0000 C CNN
+F 0 "SW3" H 10725 5260 50  0000 C CNN
 F 1 "SW_SPDT" H 10725 5169 50  0000 C CNN
 F 2 "" H 10725 4975 50  0001 C CNN
@@
 	2450 4700 2450 2900
 $Comp
-L ram-rom-upgrade-symbols:BarGraphLED_8P BAR?
+L ram-rom-upgrade-symbols:BarGraphLED_8P BAR1
 U 1 1 6086E85F
 P 4075 6850
-F 0 "BAR?" V 4075 6225 50  0000 L CNN
+F 0 "BAR1" V 4075 6225 50  0000 L CNN
 F 1 "BarGraphLED_8P" V 4120 7380 50  0001 L CNN
 F 2 "" H 4075 6850 50  0001 C CNN
@@
 $EndComp
 $Comp
-L ram-rom-upgrade-symbols:BarGraphLED_8P BAR?
+L ram-rom-upgrade-symbols:BarGraphLED_8P BAR2
 U 1 1 608742C3
 P 5075 6850
-F 0 "BAR?" V 5075 7400 50  0000 L CNN
+F 0 "BAR2" V 5075 7400 50  0000 L CNN
 F 1 "BarGraphLED_8P" V 5120 7380 50  0001 L CNN
 F 2 "" H 5075 6850 50  0001 C CNN
@@
 	2375 6450 2375 5750
 $Comp
-L Device:R_Network08_US RN?
+L Device:R_Network08_US RN1
 U 1 1 608F7760
 P 4075 7250
-F 0 "RN?" H 4600 7250 50  0000 R CNN
+F 0 "RN1" H 4600 7250 50  0000 R CNN
 F 1 "R_Network08_US" H 3595 7295 50  0001 R CNN
 F 2 "Resistor_THT:R_Array_SIP9" V 4550 7250 50  0001 C CNN
@@
 $EndComp
 $Comp
-L Device:R_Network08_US RN?
+L Device:R_Network08_US RN2
 U 1 1 608FA03A
 P 5075 7250
-F 0 "RN?" H 4600 7250 50  0000 R CNN
+F 0 "RN2" H 4600 7250 50  0000 R CNN
 F 1 "R_Network08_US" H 4595 7295 50  0001 R CNN
 F 2 "Resistor_THT:R_Array_SIP9" V 5550 7250 50  0001 C CNN
@@
 $EndComp
 $Comp
-L power:GND #PWR?
+L power:GND #PWR05
 U 1 1 608FB857
 P 4475 7450
-F 0 "#PWR?" H 4475 7200 50  0001 C CNN
+F 0 "#PWR05" H 4475 7200 50  0001 C CNN
 F 1 "GND" H 4480 7277 50  0000 C CNN
 F 2 "" H 4475 7450 50  0001 C CNN
@@
 $EndComp
 $Comp
-L power:GND #PWR?
+L power:GND #PWR06
 U 1 1 608FBDA6
 P 5475 7450
-F 0 "#PWR?" H 5475 7200 50  0001 C CNN
+F 0 "#PWR06" H 5475 7200 50  0001 C CNN
 F 1 "GND" H 5480 7277 50  0000 C CNN
 F 2 "" H 5475 7450 50  0001 C CNN
@@
 	7525 625  7250 625
 $Comp
-L power:GND #PWR?
+L power:GND #PWR09
 U 1 1 60809B64
 P 7250 625
-F 0 "#PWR?" H 7250 375 50  0001 C CNN
+F 0 "#PWR09" H 7250 375 50  0001 C CNN
 F 1 "GND" H 7255 452 50  0000 C CNN
 F 2 "" H 7250 625 50  0001 C CNN
@@
 	8675 625  7525 625
 $Comp
-L Device:R_Network08_US RN?
+L Device:R_Network08_US RN3
 U 1 1 6073A7C3
 P 7925 825
-F 0 "RN?" H 8313 871 50  0000 L CNN
+F 0 "RN3" H 8313 871 50  0000 L CNN
 F 1 "10K" H 8313 780 50  0000 L CNN
 F 2 "Resistor_THT:R_Array_SIP9" V 8400 825 50  0001 C CNN
@@
 $EndComp
 $Comp
-L Device:R_Network08_US RN?
+L Device:R_Network08_US RN4
 U 1 1 60736850
 P 9075 825
-F 0 "RN?" H 9463 871 50  0000 L CNN
+F 0 "RN4" H 9463 871 50  0000 L CNN
 F 1 "10K" H 9463 780 50  0000 L CNN
 F 2 "Resistor_THT:R_Array_SIP9" V 9550 825 50  0001 C CNN
