File: ram-rom-upgrade/schematics/address-register-16bit/address-register-16bit.sch (KiCad schematic (older format))
At the start: 14 parts

Commit message: candidate final schematic designs
Also started to consolidate custom symbols from all projects
Parts:
- BAR? (x2): symbol ram-rom-upgrade-symbols:BarGraphLED_8P -> common-symbols:BarGraphLED_8P
Changed lines of the file:
@@
 Connection ~ 2750 4300
 $Comp
-L ram-rom-upgrade-symbols:BarGraphLED_8P BAR?
+L common-symbols:BarGraphLED_8P BAR?
 U 1 1 606FFA03
 P 4825 4750
@@
 $EndComp
 $Comp
-L ram-rom-upgrade-symbols:BarGraphLED_8P BAR?
+L common-symbols:BarGraphLED_8P BAR?
 U 1 1 607039DE
 P 5800 4750
