File: instruction-register-8-bit/schematics/ram-rom-module/ram-rom-module.sch (KiCad schematic (older format))
At the start: 17 parts, among them SW1 SW_DIP_x08, SW2 SW_Push, U1 74LS245, U2 UM61512A, U3 74LS04, U4 28C256, U5 74LS257, U6 74LS157, U7 74LS00, U8 74LS32, U9 74LS257

Commit message: candidate final schematic designs
Also started to consolidate custom symbols from all projects
Parts:
- removed U7: 74LS00, symbol 74xx:74LS00
- added U? (x3): 74LS08, symbol 74xx:74LS08
- added U?: 74LS32, symbol 74xx:74LS32
- added U? (x4): 74LS04, symbol 74xx:74LS04
Connections:
- net labels added: A16, MDi, MDo, RAMe, ~ROMe
- net labels removed: A15, RMi, ~RMo
- wire segments 298 -> 293
Other:
- note removed: "Use one of the extra inverters\nfrom the program counter build."
Changed lines of the file:
@@
 encoding utf-8
 Sheet 1 1
-Title "32K RAM / 32K ROM Module for Eater SAP-1"
+Title "32K RAM / 32K ROM Module v1.1"
 Date ""
 Rev ""
@@
 A14
 Text HLabel 3025 900  1    50   Input ~ 0
-A15
+A16
 Wire Wire Line
 	1525 900  1525 1750
@@
 Wire Wire Line
 	2925 900  2925 1050
-Wire Wire Line
-	3025 900  3025 1000
-Wire Wire Line
-	3025 1000 3200 1000
-Wire Wire Line
-	3200 1000 3200 1850
 Wire Wire Line
 	2925 1050 4975 1050
@@
 Wire Wire Line
 	3300 1850 3300 1800
-Wire Wire Line
-	3025 1850 3025 1800
-Wire Wire Line
-	3025 1800 3300 1800
 Wire Wire Line
 	4350 850  4350 1875
@@
 	9700 3275 9850 3275
 $Comp
-L 74xx:74LS00 U7
-U 1 1 60A34B20
-P 9900 3875
-F 0 "U7" H 10000 3600 50  0000 R CNN
-F 1 "74LS00" H 10000 3675 50  0000 R CNN
-F 2 "" H 9900 3875 50  0001 C CNN
-F 3 "http://www.ti.com/lit/gpn/sn74ls00" H 9900 3875 50  0001 C CNN
-	1    9900 3875
-	-1   0    0    1
-$EndComp
-$Comp
-L 74xx:74LS00 U7
-U 4 1 60A61832
-P 7975 750
-F 0 "U7" H 7950 1025 50  0000 R CNN
-F 1 "74LS00" H 8075 950 50  0000 R CNN
-F 2 "" H 7975 750 50  0001 C CNN
-F 3 "http://www.ti.com/lit/gpn/sn74ls00" H 7975 750 50  0001 C CNN
-	4    7975 750
-	-1   0    0    1
-$EndComp
-$Comp
 L Device:C C1
 U 1 1 60AC7A75
@@
 $EndComp
 $Comp
-L 74xx:74LS00 U7
-U 2 1 60A3B14B
-P 9300 3875
-F 0 "U7" H 9400 3600 50  0000 R CNN
-F 1 "74LS00" H 9400 3675 50  0000 R CNN
-F 2 "" H 9300 3875 50  0001 C CNN
-F 3 "http://www.ti.com/lit/gpn/sn74ls00" H 9300 3875 50  0001 C CNN
-	2    9300 3875
-	-1   0    0    1
-$EndComp
-$Comp
 L Device:D_Schottky D1
 U 1 1 60ACD153
@@
 CLK
 Wire Wire Line
-	10200 3975 10250 3975
+	10125 3975 10200 3975
 Wire Wire Line
 	10550 3975 10600 3975
-Text HLabel 10950 3775 2    50   Input ~ 0
-RMi
+Text HLabel 10725 3475 2    50   Input ~ 0
+MDi
 Wire Wire Line
 	4675 1925 4675 1800
@@
 Wire Wire Line
 	3825 4250 3825 3800
-Text HLabel 10950 5200 2    50   Input ~ 0
-~RMo
+Text HLabel 10675 5300 2    50   Input ~ 0
+MDo
 $Comp
 L power:GND #PWR0113
@@
 	-1   0    0    1
 $EndComp
-Connection ~ 3200 1000
-Wire Wire Line
-	4575 1000 4575 1925
 Text Notes 6475 1275 0    39   ~ 0
 NOTE: This OR gate prevents the ROM & RAM \nfrom outputing to the bus if the 74LS157s are\nactive. The 74LS157s are active if RMi or the \nmanual memory write buttons are high.
@@
 	7575 3200 5675 3200
 Wire Wire Line
-	3200 1000 4575 1000
-Wire Wire Line
 	6575 2325 7075 2325
 Wire Wire Line
@@
 Wire Wire Line
 	10900 3975 10950 3975
-Wire Wire Line
-	10550 3775 10950 3775
-$Comp
-L 74xx:74LS00 U7
-U 3 1 60BCC7C3
-P 8275 5400
-F 0 "U7" H 8275 5083 50  0000 C CNN
-F 1 "74LS00" H 8275 5174 50  0000 C CNN
-F 2 "" H 8275 5400 50  0001 C CNN
-F 3 "http://www.ti.com/lit/gpn/sn74ls00" H 8275 5400 50  0001 C CNN
-	3    8275 5400
-	-1   0    0    1
-$EndComp
 Connection ~ 7975 5400
 Wire Wire Line
@@
 Wire Wire Line
 	7850 4250 8575 4250
-Wire Wire Line
-	8575 4250 8575 5300
 Connection ~ 6850 1800
 Wire Wire Line
-	8575 5300 8575 5500
-Connection ~ 8575 5300
-Wire Wire Line
-	3025 1800 1100 1800
-Wire Wire Line
 	1100 1800 1100 2325
-Connection ~ 3025 1800
 Connection ~ 1100 2325
 Wire Wire Line
-	9600 3875 9600 3775
-Wire Wire Line
-	9600 3875 9600 3975
-Connection ~ 9600 3875
-Wire Wire Line
-	10550 3775 10200 3775
-Connection ~ 10550 3775
-Wire Wire Line
-	10200 3975 10200 4275
-Connection ~ 10200 3975
-Wire Wire Line
-	9000 3575 9000 3875
-Wire Wire Line
-	10950 5200 8875 5200
-Wire Wire Line
 	8875 5200 8875 3800
 Wire Wire Line
-	3825 3800 8875 3800
-Wire Wire Line
 	8975 3275 9300 3275
 Wire Wire Line
-	10550 1575 10550 3775
+	10125 1575 10125 3375
 Wire Wire Line
 	2825 6300 4650 6300
@@
 Connection ~ 8975 3275
 Wire Wire Line
-	8275 3575 8275 2825
-Wire Wire Line
-	8275 3575 9000 3575
+	8275 3375 8275 2825
+Wire Wire Line
+	8275 3375 9225 3375
 $Comp
 L power:VCC #PWR02
@@
 	8750 3025 8750 5650
 Wire Wire Line
-	8275 850  8275 1375
-Wire Wire Line
-	8275 850  8275 650
-Connection ~ 8275 850
-Wire Wire Line
 	7675 750  6275 750
 Wire Wire Line
@@
 	6275 950  3525 950
 Wire Wire Line
-	7450 1575 10550 1575
+	7450 1575 10125 1575
 Wire Wire Line
 	7450 1375 8275 1375
@@
 $EndComp
 Wire Wire Line
-	3200 1000 3200 750
-Wire Wire Line
 	3800 750  3800 1800
 Wire Wire Line
@@
 Wire Wire Line
 	3425 1800 3425 1850
-Text Notes 3425 625  0    39   ~ 0
-Use one of the extra inverters\nfrom the program counter build.
+Wire Wire Line
+	1100 1800 3300 1800
+Wire Wire Line
+	3025 900  3025 1850
+Text HLabel 3200 550  0    50   Input ~ 0
+RAMe
+Wire Wire Line
+	3200 550  3200 750
+Connection ~ 3200 750
+Wire Wire Line
+	3200 750  3200 1850
+Text HLabel 4575 550  0    50   Input ~ 0
+~ROMe
+Wire Wire Line
+	4575 550  4575 1925
+$Comp
+L 74xx:74LS08 U?
+U 1 1 612A95F0
+P 9825 3875
+F 0 "U?" H 9825 3558 50  0000 C CNN
+F 1 "74LS08" H 9825 3649 50  0000 C CNN
+F 2 "" H 9825 3875 50  0001 C CNN
+F 3 "http://www.ti.com/lit/gpn/sn74LS08" H 9825 3875 50  0001 C CNN
+	1    9825 3875
+	-1   0    0    1
+$EndComp
+$Comp
+L 74xx:74LS32 U?
+U 1 1 612AF4C7
+P 9775 5100
+F 0 "U?" H 9775 4783 50  0000 C CNN
+F 1 "74LS32" H 9775 4874 50  0000 C CNN
+F 2 "" H 9775 5100 50  0001 C CNN
+F 3 "http://www.ti.com/lit/gpn/sn74LS32" H 9775 5100 50  0001 C CNN
+	1    9775 5100
+	-1   0    0    1
+$EndComp
+Wire Wire Line
+	9475 5300 10675 5300
+Text HLabel 10675 5000 2    50   Input ~ 0
+~ROMe
+Text HLabel 10675 5200 2    50   Input ~ 0
+RAMe
+$Comp
+L 74xx:74LS04 U?
+U 2 1 61302864
+P 10375 5000
+F 0 "U?" H 10475 5100 50  0000 C CNN
+F 1 "74LS04" H 10475 4850 50  0000 C CNN
+F 2 "" H 10375 5000 50  0001 C CNN
+F 3 "http://www.ti.com/lit/gpn/sn74LS04" H 10375 5000 50  0001 C CNN
+	2    10375 5000
+	-1   0    0    1
+$EndComp
+Wire Wire Line
+	10675 5200 10075 5200
+$Comp
+L 74xx:74LS08 U?
+U 2 1 613AB45A
+P 10425 3375
+F 0 "U?" H 10425 3058 50  0000 C CNN
+F 1 "74LS08" H 10425 3149 50  0000 C CNN
+F 2 "" H 10425 3375 50  0001 C CNN
+F 3 "http://www.ti.com/lit/gpn/sn74LS08" H 10425 3375 50  0001 C CNN
+	2    10425 3375
+	-1   0    0    1
+$EndComp
+Connection ~ 10125 3375
+Wire Wire Line
+	10125 3375 10125 3775
+Text HLabel 10725 3275 2    50   Input ~ 0
+RAMe
+Wire Wire Line
+	10200 4275 10200 3975
+Connection ~ 10200 3975
+Wire Wire Line
+	10200 3975 10250 3975
+$Comp
+L 74xx:74LS04 U?
+U 3 1 61E7E335
+P 8325 3800
+F 0 "U?" H 8425 3925 50  0000 C CNN
+F 1 "74LS04" H 8475 3675 50  0000 C CNN
+F 2 "" H 8325 3800 50  0001 C CNN
+F 3 "http://www.ti.com/lit/gpn/sn74LS04" H 8325 3800 50  0001 C CNN
+	3    8325 3800
+	-1   0    0    1
+$EndComp
+$Comp
+L 74xx:74LS04 U?
+U 4 1 61E81919
+P 7975 750
+F 0 "U?" H 8050 875 50  0000 C CNN
+F 1 "74LS04" H 8100 625 50  0000 C CNN
+F 2 "" H 7975 750 50  0001 C CNN
+F 3 "http://www.ti.com/lit/gpn/sn74LS04" H 7975 750 50  0001 C CNN
+	4    7975 750
+	-1   0    0    1
+$EndComp
+Wire Wire Line
+	8275 750  8275 1375
+$Comp
+L 74xx:74LS04 U?
+U 5 1 61E9D82B
+P 8275 5400
+F 0 "U?" H 8275 5083 50  0000 C CNN
+F 1 "74LS04" H 8275 5174 50  0000 C CNN
+F 2 "" H 8275 5400 50  0001 C CNN
+F 3 "http://www.ti.com/lit/gpn/sn74LS04" H 8275 5400 50  0001 C CNN
+	5    8275 5400
+	-1   0    0    1
+$EndComp
+Wire Wire Line
+	8575 4250 8575 5400
+Wire Wire Line
+	9525 3875 9225 3875
+Wire Wire Line
+	9225 3375 9225 3875
+$Comp
+L 74xx:74LS08 U?
+U 4 1 61ED6FDD
+P 9175 5200
+F 0 "U?" H 9175 4883 50  0000 C CNN
+F 1 "74LS08" H 9175 4974 50  0000 C CNN
+F 2 "" H 9175 5200 50  0001 C CNN
+F 3 "http://www.ti.com/lit/gpn/sn74LS08" H 9175 5200 50  0001 C CNN
+	4    9175 5200
+	-1   0    0    1
+$EndComp
+Wire Wire Line
+	8875 3800 8625 3800
+Wire Wire Line
+	8025 3800 3825 3800
 $EndSCHEMATC

Commit message: removed A16 address line
Parts:
- gave numbers to parts that had none: 3
- renumbered R2 to R1, R1 to R2, U3 to U2, U2 to U3, U5 to U4, U4 to U5, U8 to U6, U9 to U7, U6 to U8
Changed lines of the file:
@@
 $EndDescr
 $Comp
-L common-symbols:UM61512A U2
+L common-symbols:UM61512A U3
 U 1 1 6042600F
 P 3650 1950
-F 0 "U2" V 4450 -250 50  0000 C CNN
+F 0 "U3" V 4450 -250 50  0000 C CNN
 F 1 "UM61512A" V 4000 775 50  0000 C CNN
 F 2 "" H 3900 -150 50  0001 C CNN
@@
 	1575 4475 1575 4550
 $Comp
-L power:GND #PWR0101
+L power:GND #PWR02
 U 1 1 605DD0AA
 P 1575 5025
-F 0 "#PWR0101" H 1575 4775 50  0001 C CNN
+F 0 "#PWR02" H 1575 4775 50  0001 C CNN
 F 1 "GND" H 1580 4852 50  0000 C CNN
 F 2 "" H 1575 5025 50  0001 C CNN
@@
 	4350 5300 4350 6475
 $Comp
-L Memory_EEPROM:28C256 U4
+L Memory_EEPROM:28C256 U5
 U 1 1 606B59F6
 P 5475 2325
-F 0 "U4" V 5825 1325 50  0000 L CNN
+F 0 "U5" V 5825 1325 50  0000 L CNN
 F 1 "28C256" V 5450 2175 50  0000 L CNN
 F 2 "" H 5475 2325 50  0001 C CNN
@@
 	1525 1750 1525 1850
 $Comp
-L power:GND #PWR0102
+L power:GND #PWR04
 U 1 1 6081049F
 P 4100 2325
-F 0 "#PWR0102" H 4100 2075 50  0001 C CNN
+F 0 "#PWR04" H 4100 2075 50  0001 C CNN
 F 1 "GND" H 4105 2152 50  0000 C CNN
 F 2 "" H 4100 2325 50  0001 C CNN
@@
 $EndComp
 $Comp
-L power:VCC #PWR0103
+L power:VCC #PWR06
 U 1 1 60810E8E
 P 4350 850
-F 0 "#PWR0103" H 4350 700 50  0001 C CNN
+F 0 "#PWR06" H 4350 700 50  0001 C CNN
 F 1 "VCC" H 4365 1023 50  0000 C CNN
 F 2 "" H 4350 850 50  0001 C CNN
@@
 	4350 850  4350 1875
 $Comp
-L power:GND #PWR0104
+L power:GND #PWR09
 U 1 1 608E68AE
 P 6250 4750
-F 0 "#PWR0104" H 6250 4500 50  0001 C CNN
+F 0 "#PWR09" H 6250 4500 50  0001 C CNN
 F 1 "GND" H 6255 4577 50  0000 C CNN
 F 2 "" H 6250 4750 50  0001 C CNN
@@
 $EndComp
 $Comp
-L power:GND #PWR0105
+L power:GND #PWR013
 U 1 1 608F4888
 P 8275 4750
-F 0 "#PWR0105" H 8275 4500 50  0001 C CNN
+F 0 "#PWR013" H 8275 4500 50  0001 C CNN
 F 1 "GND" H 8280 4577 50  0000 C CNN
 F 2 "" H 8275 4750 50  0001 C CNN
@@
 	3525 1850 3525 950
 $Comp
-L 74xx:74LS157 U6
+L 74xx:74LS157 U8
 U 1 1 6091C4A7
 P 7975 2325
-F 0 "U6" V 7700 3175 50  0000 R CNN
+F 0 "U8" V 7700 3175 50  0000 R CNN
 F 1 "74LS157" V 8000 2475 50  0000 R CNN
 F 2 "" H 7975 2325 50  0001 C CNN
@@
 PROG
 $Comp
-L Device:R_Small R2
+L Device:R_Small R1
 U 1 1 609DB4E4
 P 8975 3025
-F 0 "R2" V 9050 2975 50  0000 L CNN
+F 0 "R1" V 9050 2975 50  0000 L CNN
 F 1 "1K Ω" V 8900 2925 50  0000 L CNN
 F 2 "" H 8975 3025 50  0001 C CNN
@@
 	8975 3125 8975 3275
 $Comp
-L power:GND #PWR0106
+L power:GND #PWR014
 U 1 1 60A080BD
 P 9150 2325
-F 0 "#PWR0106" H 9150 2075 50  0001 C CNN
+F 0 "#PWR014" H 9150 2075 50  0001 C CNN
 F 1 "GND" H 9155 2152 50  0000 C CNN
 F 2 "" H 9150 2325 50  0001 C CNN
@@
 $EndComp
 $Comp
-L power:VCC #PWR0107
+L power:VCC #PWR015
 U 1 1 60A087AA
 P 9850 3275
-F 0 "#PWR0107" H 9850 3125 50  0001 C CNN
+F 0 "#PWR015" H 9850 3125 50  0001 C CNN
 F 1 "VCC" H 9865 3448 50  0000 C CNN
 F 2 "" H 9850 3275 50  0001 C CNN
@@
 $EndComp
 $Comp
-L Device:R_Small R1
+L Device:R_Small R2
 U 1 1 60ACDD52
 P 10200 4375
-F 0 "R1" V 10275 4325 50  0000 L CNN
+F 0 "R2" V 10275 4325 50  0000 L CNN
 F 1 "1K Ω" V 10125 4275 50  0000 L CNN
 F 2 "" H 10200 4375 50  0001 C CNN
@@
 $EndComp
 $Comp
-L power:GND #PWR0108
+L power:GND #PWR016
 U 1 1 60ACF243
 P 10200 4475
-F 0 "#PWR0108" H 10200 4225 50  0001 C CNN
+F 0 "#PWR016" H 10200 4225 50  0001 C CNN
 F 1 "GND" H 10205 4302 50  0000 C CNN
 F 2 "" H 10200 4475 50  0001 C CNN
@@
 Connection ~ 4650 3725
 $Comp
-L power:VCC #PWR0109
+L power:VCC #PWR07
 U 1 1 60C15423
 P 4350 4750
-F 0 "#PWR0109" H 4350 4600 50  0001 C CNN
+F 0 "#PWR07" H 4350 4600 50  0001 C CNN
 F 1 "VCC" H 4365 4923 50  0000 C CNN
 F 2 "" H 4350 4750 50  0001 C CNN
@@
 	3850 7150 3950 7150
 $Comp
-L power:GND #PWR0110
+L power:GND #PWR08
 U 1 1 60CD7BF0
 P 4450 7250
-F 0 "#PWR0110" H 4450 7000 50  0001 C CNN
+F 0 "#PWR08" H 4450 7000 50  0001 C CNN
 F 1 "GND" H 4455 7077 50  0000 C CNN
 F 2 "" H 4450 7250 50  0001 C CNN
@@
 NoConn ~ 7375 1825
 $Comp
-L power:GND #PWR0111
+L power:GND #PWR012
 U 1 1 60D9C95B
 P 8075 2950
-F 0 "#PWR0111" H 8075 2700 50  0001 C CNN
+F 0 "#PWR012" H 8075 2700 50  0001 C CNN
 F 1 "GND" H 8080 2777 50  0000 C CNN
 F 2 "" H 8075 2950 50  0001 C CNN
@@
 Connection ~ 8075 2875
 $Comp
-L power:VCC #PWR0112
+L power:VCC #PWR011
 U 1 1 60F054EC
 P 7075 2200
-F 0 "#PWR0112" H 7075 2050 50  0001 C CNN
+F 0 "#PWR011" H 7075 2050 50  0001 C CNN
 F 1 "VCC" H 7090 2373 50  0000 C CNN
 F 2 "" H 7075 2200 50  0001 C CNN
@@
 MDo
 $Comp
-L power:GND #PWR0113
+L power:GND #PWR05
 U 1 1 60F70DD4
 P 4125 4750
-F 0 "#PWR0113" H 4125 4500 50  0001 C CNN
+F 0 "#PWR05" H 4125 4500 50  0001 C CNN
 F 1 "GND" H 4130 4577 50  0000 C CNN
 F 2 "" H 4125 4750 50  0001 C CNN
@@
 $EndComp
 $Comp
-L power:GND #PWR0114
+L power:GND #PWR01
 U 1 1 60F871F3
 P 1100 2550
-F 0 "#PWR0114" H 1100 2300 50  0001 C CNN
+F 0 "#PWR01" H 1100 2300 50  0001 C CNN
 F 1 "GND" H 1105 2377 50  0000 C CNN
 F 2 "" H 1100 2550 50  0001 C CNN
@@
 	7975 5400 7975 5250
 $Comp
-L 74xx:74LS32 U8
+L 74xx:74LS32 U6
 U 1 1 60819261
 P 7150 1475
-F 0 "U8" H 7075 1750 50  0000 C CNN
+F 0 "U6" H 7075 1750 50  0000 C CNN
 F 1 "74LS32" H 7150 1675 50  0000 C CNN
 F 2 "" H 7150 1475 50  0001 C CNN
@@
 	8275 3375 9225 3375
 $Comp
-L power:VCC #PWR02
+L power:VCC #PWR010
 U 1 1 60A653A0
 P 6375 4750
-F 0 "#PWR02" H 6375 4600 50  0001 C CNN
+F 0 "#PWR010" H 6375 4600 50  0001 C CNN
 F 1 "VCC" H 6390 4923 50  0000 C CNN
 F 2 "" H 6375 4750 50  0001 C CNN
@@
 $EndComp
 $Comp
-L power:VCC #PWR01
+L power:VCC #PWR03
 U 1 1 60A65B45
 P 2525 4175
-F 0 "#PWR01" H 2525 4025 50  0001 C CNN
+F 0 "#PWR03" H 2525 4025 50  0001 C CNN
 F 1 "VCC" H 2540 4348 50  0000 C CNN
 F 2 "" H 2525 4175 50  0001 C CNN
@@
 	8275 1375 8275 1825
 $Comp
-L common-symbols:74LS257 U9
+L common-symbols:74LS257 U7
 U 1 1 607C5143
 P 7275 4750
-F 0 "U9" V 7525 3925 50  0000 R CNN
+F 0 "U7" V 7525 3925 50  0000 R CNN
 F 1 "74LS257" V 7275 4900 50  0000 R CNN
 F 2 "" H 7275 4750 50  0001 C CNN
@@
 $EndComp
 $Comp
-L common-symbols:74LS257 U5
+L common-symbols:74LS257 U4
 U 1 1 60814B6F
 P 5250 4750
-F 0 "U5" V 5500 3925 50  0000 R CNN
+F 0 "U4" V 5500 3925 50  0000 R CNN
 F 1 "74LS257" V 5250 4900 50  0000 R CNN
 F 2 "" H 5250 4750 50  0001 C CNN
@@
 $EndComp
 $Comp
-L 74xx:74LS04 U3
+L 74xx:74LS04 U2
 U 1 1 60BA129D
 P 3500 750
-F 0 "U3" H 3450 750 50  0000 C CNN
+F 0 "U2" H 3450 750 50  0000 C CNN
 F 1 "74LS04" H 3500 976 50  0001 C CNN
 F 2 "" H 3500 750 50  0001 C CNN
@@
 	4575 550  4575 1925
 $Comp
-L 74xx:74LS08 U?
+L 74xx:74LS08 U9
 U 1 1 612A95F0
 P 9825 3875
-F 0 "U?" H 9825 3558 50  0000 C CNN
+F 0 "U9" H 9825 3558 50  0000 C CNN
 F 1 "74LS08" H 9825 3649 50  0000 C CNN
 F 2 "" H 9825 3875 50  0001 C CNN
@@
 $EndComp
 $Comp
-L 74xx:74LS32 U?
+L 74xx:74LS32 U10
 U 1 1 612AF4C7
 P 9775 5100
-F 0 "U?" H 9775 4783 50  0000 C CNN
+F 0 "U10" H 9775 4783 50  0000 C CNN
 F 1 "74LS32" H 9775 4874 50  0000 C CNN
 F 2 "" H 9775 5100 50  0001 C CNN
@@
 RAMe
 $Comp
-L 74xx:74LS04 U?
+L 74xx:74LS04 U2
 U 2 1 61302864
 P 10375 5000
-F 0 "U?" H 10475 5100 50  0000 C CNN
+F 0 "U2" H 10475 5100 50  0000 C CNN
 F 1 "74LS04" H 10475 4850 50  0000 C CNN
 F 2 "" H 10375 5000 50  0001 C CNN
@@
 	10675 5200 10075 5200
 $Comp
-L 74xx:74LS08 U?
+L 74xx:74LS08 U9
 U 2 1 613AB45A
 P 10425 3375
-F 0 "U?" H 10425 3058 50  0000 C CNN
+F 0 "U9" H 10425 3058 50  0000 C CNN
 F 1 "74LS08" H 10425 3149 50  0000 C CNN
 F 2 "" H 10425 3375 50  0001 C CNN
@@
 	10200 3975 10250 3975
 $Comp
-L 74xx:74LS04 U?
+L 74xx:74LS04 U2
 U 3 1 61E7E335
 P 8325 3800
-F 0 "U?" H 8425 3925 50  0000 C CNN
+F 0 "U2" H 8425 3925 50  0000 C CNN
 F 1 "74LS04" H 8475 3675 50  0000 C CNN
 F 2 "" H 8325 3800 50  0001 C CNN
@@
 $EndComp
 $Comp
-L 74xx:74LS04 U?
+L 74xx:74LS04 U2
 U 4 1 61E81919
 P 7975 750
-F 0 "U?" H 8050 875 50  0000 C CNN
+F 0 "U2" H 8050 875 50  0000 C CNN
 F 1 "74LS04" H 8100 625 50  0000 C CNN
 F 2 "" H 7975 750 50  0001 C CNN
@@
 	8275 750  8275 1375
 $Comp
-L 74xx:74LS04 U?
+L 74xx:74LS04 U2
 U 5 1 61E9D82B
 P 8275 5400
-F 0 "U?" H 8275 5083 50  0000 C CNN
-F 1 "74LS04" H 8275 5174 50  0000 C CNN
+F 0 "U2" H 8300 5550 50  0000 C CNN
+F 1 "74LS04" H 8350 5250 50  0000 C CNN
 F 2 "" H 8275 5400 50  0001 C CNN
 F 3 "http://www.ti.com/lit/gpn/sn74LS04" H 8275 5400 50  0001 C CNN
@@
 	9225 3375 9225 3875
 $Comp
-L 74xx:74LS08 U?
+L 74xx:74LS08 U9
 U 4 1 61ED6FDD
 P 9175 5200
-F 0 "U?" H 9175 4883 50  0000 C CNN
+F 0 "U9" H 9175 4883 50  0000 C CNN
 F 1 "74LS08" H 9175 4974 50  0000 C CNN
 F 2 "" H 9175 5200 50  0001 C CNN
