File: instruction-register-8-bit/schematics/run-mode-selector-16bit/run-mode-selector-16bit.sch (KiCad schematic (older format))
At the start: 19 parts, among them SW1 SW_DIP_x08, SW2 SW_DIP_x08, SW3 SW_SPDT, U1 74LS157, U2 74LS157, U3 74LS157, U4 74LS157

Commit message: removed A16 address line
Parts:
- removed R?: 1K, symbol Device:R
- BAR1, BAR2: symbol ram-rom-upgrade-symbols:BarGraphLED_8P -> common-symbols:BarGraphLED_8P
Changed lines of the file:
@@
 	2450 3025 2450 1225
 $Comp
-L ram-rom-upgrade-symbols:BarGraphLED_8P BAR1
+L common-symbols:BarGraphLED_8P BAR1
 U 1 1 6086E85F
 P 4075 5175
@@
 $EndComp
 $Comp
-L ram-rom-upgrade-symbols:BarGraphLED_8P BAR2
+L common-symbols:BarGraphLED_8P BAR2
 U 1 1 608742C3
 P 5075 5175
@@
 Wire Wire Line
 	2450 4100 2450 7500
-Text HLabel 2075 7500 3    50   Output ~ 0
-A16
-$Comp
-L power:GND #PWR?
-U 1 1 61F7ADFA
-P 1575 7375
-F 0 "#PWR?" H 1575 7125 50  0001 C CNN
-F 1 "GND" H 1580 7202 50  0000 C CNN
-F 2 "" H 1575 7375 50  0001 C CNN
-F 3 "" H 1575 7375 50  0001 C CNN
-	1    1575 7375
-	1    0    0    -1
-$EndComp
-$Comp
-L Device:R R?
-U 1 1 61F7B8D9
-P 1825 7375
-F 0 "R?" V 1750 7375 50  0000 C CNN
-F 1 "1K" V 1825 7375 50  0000 C CNN
-F 2 "" V 1755 7375 50  0001 C CNN
-F 3 "~" H 1825 7375 50  0001 C CNN
-	1    1825 7375
-	0    1    1    0
-$EndComp
-Wire Wire Line
-	1975 7375 2075 7375
-Wire Wire Line
-	2075 7375 2075 7500
-Wire Wire Line
-	1675 7375 1575 7375
 $EndSCHEMATC

Commit message: seperated RAM and ROM modules
In order to simplify each, the RAM and ROM modules are seperated and no longer share a common connection to the data bus. Also added support for addres line A16, though it is tied to ground and outherwise unused in this design
Parts:
- added R?: 1K, symbol Device:R
Connections:
- net GND: now also R?.1
- new net A16: R?.2
Changed lines of the file:
@@
 Wire Wire Line
 	2450 4100 2450 7500
+Text HLabel 2075 7500 3    50   Output ~ 0
+A16
+$Comp
+L power:GND #PWR?
+U 1 1 6105A225
+P 1650 7325
+F 0 "#PWR?" H 1650 7075 50  0001 C CNN
+F 1 "GND" H 1655 7152 50  0000 C CNN
+F 2 "" H 1650 7325 50  0001 C CNN
+F 3 "" H 1650 7325 50  0001 C CNN
+	1    1650 7325
+	1    0    0    -1
+$EndComp
+$Comp
+L Device:R R?
+U 1 1 6105B7B2
+P 1925 7325
+F 0 "R?" V 2000 7325 50  0000 C CNN
+F 1 "1K" V 1925 7325 50  0000 C CNN
+F 2 "" V 1855 7325 50  0001 C CNN
+F 3 "~" H 1925 7325 50  0001 C CNN
+	1    1925 7325
+	0    -1   -1   0
+$EndComp
+Wire Wire Line
+	2075 7500 2075 7325
+Wire Wire Line
+	1775 7325 1650 7325
 $EndSCHEMATC
