File: instruction-register-8-bit/schematics/rom-module/rom-module.sch (KiCad schematic (older format))
At the start: 7 parts

Commit message: updated annotations
Parts:
- gave numbers to parts that had none: 6
Changed lines of the file:
@@
 $EndDescr
 $Comp
-L Memory_EEPROM:28C256 U?
+L Memory_EEPROM:28C256 U3
 U 1 1 612FE2F8
 P 5625 2900
-F 0 "U?" V 5875 3925 50  0000 L CNN
+F 0 "U3" V 5875 3925 50  0000 L CNN
 F 1 "28C256" V 5625 2750 50  0000 L CNN
 F 2 "" H 5625 2900 50  0001 C CNN
@@
 $EndComp
 $Comp
-L 74xx:74LS245 U?
+L 74xx:74LS245 U4
 U 1 1 6130142A
 P 6025 5075
-F 0 "U?" V 5979 5919 50  0000 L CNN
+F 0 "U4" V 5979 5919 50  0000 L CNN
 F 1 "74LS245" V 6070 5919 50  0000 L CNN
 F 2 "" H 6025 5075 50  0001 C CNN
@@
 	5125 2500 5125 2100
 $Comp
-L 74xx:74LS08 U?
+L 74xx:74LS08 U2
 U 1 1 6131C20E
 P 2650 3875
-F 0 "U?" H 2650 4200 50  0000 C CNN
+F 0 "U2" H 2650 4200 50  0000 C CNN
 F 1 "74LS08" H 2650 4109 50  0000 C CNN
 F 2 "" H 2650 3875 50  0001 C CNN
@@
 MDo
 $Comp
-L 74xx:74LS04 U?
+L 74xx:74LS04 U1
 U 1 1 6132310A
 P 2000 3775
-F 0 "U?" H 2000 4092 50  0000 C CNN
+F 0 "U1" H 2000 4092 50  0000 C CNN
 F 1 "74LS04" H 2000 4001 50  0000 C CNN
 F 2 "" H 2000 3775 50  0001 C CNN
@@
 	1275 3775 1500 3775
 $Comp
-L 74xx:74LS04 U?
+L 74xx:74LS04 U1
 U 2 1 61326698
 P 3325 3875
-F 0 "U?" H 3325 4192 50  0000 C CNN
+F 0 "U1" H 3325 4192 50  0000 C CNN
 F 1 "74LS04" H 3325 4101 50  0000 C CNN
 F 2 "" H 3325 3875 50  0001 C CNN
@@
 	6825 4500 6825 5075
 $Comp
-L power:VCC #PWR?
+L power:VCC #PWR04
 U 1 1 6132F6F5
 P 6825 4500
-F 0 "#PWR?" H 6825 4350 50  0001 C CNN
+F 0 "#PWR04" H 6825 4350 50  0001 C CNN
 F 1 "VCC" H 6840 4673 50  0000 C CNN
 F 2 "" H 6825 4500 50  0001 C CNN
@@
 Connection ~ 6825 4500
 $Comp
-L power:VCC #PWR?
+L power:VCC #PWR03
 U 1 1 6132F9EC
 P 6725 2425
-F 0 "#PWR?" H 6725 2275 50  0001 C CNN
+F 0 "#PWR03" H 6725 2275 50  0001 C CNN
 F 1 "VCC" H 6740 2598 50  0000 C CNN
 F 2 "" H 6725 2425 50  0001 C CNN
@@
 Connection ~ 6725 2425
 $Comp
-L power:GND #PWR?
+L power:GND #PWR01
 U 1 1 6132FD1E
 P 4525 2900
-F 0 "#PWR?" H 4525 2650 50  0001 C CNN
+F 0 "#PWR01" H 4525 2650 50  0001 C CNN
 F 1 "GND" H 4530 2727 50  0000 C CNN
 F 2 "" H 4525 2900 50  0001 C CNN
@@
 Connection ~ 4525 2900
 $Comp
-L power:GND #PWR?
+L power:GND #PWR02
 U 1 1 6133001D
 P 5225 5075
-F 0 "#PWR?" H 5225 4825 50  0001 C CNN
+F 0 "#PWR02" H 5225 4825 50  0001 C CNN
 F 1 "GND" H 5230 4902 50  0000 C CNN
 F 2 "" H 5225 5075 50  0001 C CNN
@@
 $EndComp
 $Comp
-L common-symbols:BarGraphLED_8P BAR?
+L common-symbols:BarGraphLED_8P BAR1
 U 1 1 61330C45
 P 7375 3775
-F 0 "BAR?" H 7375 4442 50  0000 C CNN
+F 0 "BAR1" H 7375 4442 50  0000 C CNN
 F 1 "BarGraphLED_8P" H 7375 4351 50  0000 C CNN
 F 2 "" H 7375 3775 50  0001 C CNN
@@
 $EndComp
 $Comp
-L Device:R_Network08 RN?
+L Device:R_Network08 RN1
 U 1 1 61333752
 P 8075 3775
-F 0 "RN?" V 7458 3775 50  0000 C CNN
+F 0 "RN1" V 7458 3775 50  0000 C CNN
 F 1 "R_Network08" V 7549 3775 50  0000 C CNN
 F 2 "Resistor_THT:R_Array_SIP9" V 8550 3775 50  0001 C CNN
@@
 $EndComp
 $Comp
-L power:GND #PWR?
+L power:GND #PWR05
 U 1 1 6133637F
 P 8425 3375
-F 0 "#PWR?" H 8425 3125 50  0001 C CNN
+F 0 "#PWR05" H 8425 3125 50  0001 C CNN
 F 1 "GND" H 8430 3202 50  0000 C CNN
 F 2 "" H 8425 3375 50  0001 C CNN
