File: stack-pointer/schematics/program-counter-16bit/program-counter-16bit.sch (KiCad schematic (older format))
At the start: 21 parts

Commit message: further work on microcode
Connections:
- net PCo renamed PCa
Changed lines of the file:
@@
 	6925 6325 6600 6325
 Text HLabel 2100 7000 0    50   Input ~ 0
-PCo
+PCa
 $Comp
 L 74xx:74LS04 U?

Commit message: added schematics to documentation
Parts:
- gave numbers to parts that had none: 17
