File: lcd-display/schematics/lcd-display/lcd-display.kicad_sch (KiCad schematic)
At the start: 13 parts, among them U1 74LS04, U2 74LS08, U3 74LS245, U4 74LS32

Commit message: addressed several stability issues
Parts:
- added C?: 22 pF, symbol Device:C
Connections:
- net GND: now also C?.1
Changed lines of the file:
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@@
+    (stroke (width 0) (type default) (color 0 0 0 0))
+  )
+  (wire (pts (xy 234.315 23.495) (xy 245.11 23.495))
     (stroke (width 0) (type default) (color 0 0 0 0))
   )
@@
     (pin "1")
   )
+  (symbol (lib_id "Device:C") (at 245.11 27.305 0) (unit 1)
+    (in_bom yes) (on_board yes) (fields_autoplaced)
+    (property "Reference" "C?" (id 0) (at 248.031 26.3965 0)
+      (effects (font (size 1.27 1.27)) (justify left))
+    )
+    (property "Value" "22 pF" (id 1) (at 248.031 29.1716 0)
+      (effects (font (size 1.27 1.27)) (justify left))
+    )
+    (property "Footprint" "" (id 2) (at 246.0752 31.115 0)
+      (effects (font (size 1.27 1.27)) hide)
+    )
+    (property "Datasheet" "~" (id 3) (at 245.11 27.305 0)
+      (effects (font (size 1.27 1.27)) hide)
+    )
+    (pin "1")
+    (pin "2")
+  )
   (symbol (lib_id "Device:C") (at 234.315 46.355 0) (unit 1)
     (in_bom yes) (on_board yes)
@@
     (pin "1")
     (pin "2")
+  )
+  (symbol (lib_id "power:GND") (at 234.315 23.495 0) (unit 1)
+    (in_bom yes) (on_board yes) (fields_autoplaced)
+    (property "Reference" "#PWR?" (id 0) (at 234.315 29.845 0)
+      (effects (font (size 1.27 1.27)) hide)
+    )
+    (property "Value" "GND" (id 1) (at 234.315 28.0575 0))
+    (property "Footprint" "" (id 2) (at 234.315 23.495 0)
+      (effects (font (size 1.27 1.27)) hide)
+    )
+    (property "Datasheet" "" (id 3) (at 234.315 23.495 0)
+      (effects (font (size 1.27 1.27)) hide)
+    )
+    (pin "1")
   )
   (sheet_instances
@@
       (reference "#PWR09") (unit 1) (value "GND") (footprint "")
     )
+    (path "/e7850ef5-b65a-428c-9e79-b5b3bf42d7ab"
+      (reference "#PWR?") (unit 1) (value "GND") (footprint "")
+    )
     (path "/00000000-0000-0000-0000-000061d87343"
       (reference "C1") (unit 1) (value "0.1 uF") (footprint "")
@@
       (reference "C7") (unit 1) (value "1 pF") (footprint "")
     )
+    (path "/0e2270f1-03a5-4a80-b6d9-892401a77bc3"
+      (reference "C?") (unit 1) (value "22 pF") (footprint "")
+    )
     (path "/00000000-0000-0000-0000-000061c95bc7"

Commit message: teweaks to design
Parts:
- added C6: 0.1 µF, symbol Device:C
- gave numbers to parts that had none: 1
- renumbered C6 to C7, C7 to C9
Connections:
- net GND: now also C6.2
- net at U1.4, U2.4: now also C6.1
Changed lines of the file:
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@@
   (junction (at 60.325 48.26) (diameter 0) (color 0 0 0 0)
   )
+  (junction (at 199.39 64.135) (diameter 0) (color 0 0 0 0)
+  )
   (junction (at 60.325 65.405) (diameter 0) (color 0 0 0 0)
   )
@@
   (junction (at 227.965 38.735) (diameter 0) (color 0 0 0 0)
   )
+  (junction (at 193.04 72.39) (diameter 0) (color 0 0 0 0)
+  )
   (junction (at 245.11 33.655) (diameter 0) (color 0 0 0 0)
   )
@@
     (stroke (width 0) (type default) (color 0 0 0 0))
   )
-  (wire (pts (xy 227.965 52.07) (xy 197.485 52.07))
+  (wire (pts (xy 227.965 52.07) (xy 196.215 52.07))
     (stroke (width 0) (type default) (color 0 0 0 0))
   )
@@
     (stroke (width 0) (type default) (color 0 0 0 0))
   )
+  (wire (pts (xy 193.04 72.39) (xy 199.39 72.39))
+    (stroke (width 0) (type default) (color 0 0 0 0))
+  )
   (wire (pts (xy 194.945 24.13) (xy 203.835 24.13))
     (stroke (width 0) (type default) (color 0 0 0 0))
@@
     (stroke (width 0) (type default) (color 0 0 0 0))
   )
-  (wire (pts (xy 175.26 64.135) (xy 210.185 64.135))
+  (wire (pts (xy 175.26 64.135) (xy 199.39 64.135))
     (stroke (width 0) (type default) (color 0 0 0 0))
   )
@@
     (stroke (width 0) (type default) (color 0 0 0 0))
   )
+  (wire (pts (xy 199.39 72.39) (xy 199.39 71.755))
+    (stroke (width 0) (type default) (color 0 0 0 0))
+  )
   (wire (pts (xy 50.8 98.425) (xy 168.91 98.425))
     (stroke (width 0) (type default) (color 0 0 0 0))
@@
     (stroke (width 0) (type default) (color 0 0 0 0))
   )
-  (wire (pts (xy 166.37 125.095) (xy 197.485 125.095))
+  (wire (pts (xy 166.37 125.095) (xy 196.215 125.095))
     (stroke (width 0) (type default) (color 0 0 0 0))
   )
@@
     (stroke (width 0) (type default) (color 0 0 0 0))
   )
+  (wire (pts (xy 199.39 64.135) (xy 210.185 64.135))
+    (stroke (width 0) (type default) (color 0 0 0 0))
+  )
   (wire (pts (xy 194.31 85.725) (xy 250.825 85.725))
     (stroke (width 0) (type default) (color 0 0 0 0))
@@
     (stroke (width 0) (type default) (color 0 0 0 0))
   )
-  (wire (pts (xy 197.485 52.07) (xy 197.485 125.095))
+  (wire (pts (xy 196.215 52.07) (xy 196.215 125.095))
     (stroke (width 0) (type default) (color 0 0 0 0))
   )
   (text "These double inverters are to ensure the\nclock signal arives after the LCD module \nhas responsed to the RS and R/W signals."
-    (at 204.47 77.47 0)
+    (at 211.455 77.47 0)
     (effects (font (size 1.4986 1.4986)) (justify left bottom))
   )
@@
   (symbol (lib_id "Device:C") (at 245.11 46.355 0) (unit 1)
     (in_bom yes) (on_board yes)
-    (property "Reference" "C7" (id 0) (at 248.031 45.1866 0)
+    (property "Reference" "C9" (id 0) (at 248.031 45.1866 0)
       (effects (font (size 1.27 1.27)) (justify left))
     )
@@
   (symbol (lib_id "power:GND") (at 245.11 50.165 0) (unit 1)
     (in_bom yes) (on_board yes)
-    (property "Reference" "#PWR09" (id 0) (at 245.11 56.515 0)
+    (property "Reference" "#PWR010" (id 0) (at 245.11 56.515 0)
       (effects (font (size 1.27 1.27)) hide)
     )
@@
   (symbol (lib_id "power:GND") (at 234.315 50.165 0) (unit 1)
     (in_bom yes) (on_board yes)
-    (property "Reference" "#PWR08" (id 0) (at 234.315 56.515 0)
+    (property "Reference" "#PWR09" (id 0) (at 234.315 56.515 0)
       (effects (font (size 1.27 1.27)) hide)
     )
@@
   (symbol (lib_id "Device:C") (at 245.11 27.305 0) (unit 1)
     (in_bom yes) (on_board yes) (fields_autoplaced)
-    (property "Reference" "C?" (id 0) (at 248.031 26.3965 0)
+    (property "Reference" "C8" (id 0) (at 248.031 26.3965 0)
       (effects (font (size 1.27 1.27)) (justify left))
     )
@@
     (pin "2")
   )
+  (symbol (lib_id "Device:C") (at 199.39 67.945 0) (unit 1)
+    (in_bom yes) (on_board yes) (fields_autoplaced)
+    (property "Reference" "C6" (id 0) (at 202.311 67.0365 0)
+      (effects (font (size 1.27 1.27)) (justify left))
+    )
+    (property "Value" "0.1 µF" (id 1) (at 202.311 69.8116 0)
+      (effects (font (size 1.27 1.27)) (justify left))
+    )
+    (property "Footprint" "" (id 2) (at 200.3552 71.755 0)
+      (effects (font (size 1.27 1.27)) hide)
+    )
+    (property "Datasheet" "~" (id 3) (at 199.39 67.945 0)
+      (effects (font (size 1.27 1.27)) hide)
+    )
+    (pin "1")
+    (pin "2")
+  )
   (symbol (lib_id "Device:C") (at 234.315 46.355 0) (unit 1)
     (in_bom yes) (on_board yes)
-    (property "Reference" "C6" (id 0) (at 237.236 45.1866 0)
+    (property "Reference" "C7" (id 0) (at 237.236 45.1866 0)
       (effects (font (size 1.27 1.27)) (justify left))
     )
@@
   (symbol (lib_id "power:GND") (at 234.315 23.495 0) (unit 1)
     (in_bom yes) (on_board yes) (fields_autoplaced)
-    (property "Reference" "#PWR?" (id 0) (at 234.315 29.845 0)
+    (property "Reference" "#PWR08" (id 0) (at 234.315 29.845 0)
       (effects (font (size 1.27 1.27)) hide)
     )
@@
       (reference "#PWR07") (unit 1) (value "GND") (footprint "")
     )
+    (path "/e7850ef5-b65a-428c-9e79-b5b3bf42d7ab"
+      (reference "#PWR08") (unit 1) (value "GND") (footprint "")
+    )
     (path "/0ae0dde3-a8f0-402c-b308-f4d09e8aaec5"
-      (reference "#PWR08") (unit 1) (value "GND") (footprint "")
+      (reference "#PWR09") (unit 1) (value "GND") (footprint "")
     )
     (path "/00000000-0000-0000-0000-000061d0faec"
-      (reference "#PWR09") (unit 1) (value "GND") (footprint "")
-    )
-    (path "/e7850ef5-b65a-428c-9e79-b5b3bf42d7ab"
-      (reference "#PWR?") (unit 1) (value "GND") (footprint "")
+      (reference "#PWR010") (unit 1) (value "GND") (footprint "")
     )
     (path "/00000000-0000-0000-0000-000061d87343"
@@
       (reference "C5") (unit 1) (value "0.1 uF") (footprint "")
     )
+    (path "/2f40c2ed-ea77-481a-b728-3e9572b94a99"
+      (reference "C6") (unit 1) (value "0.1 µF") (footprint "")
+    )
     (path "/9a7ade3c-a81d-4038-a57c-b220b9c3cd90"
-      (reference "C6") (unit 1) (value "1 pF") (footprint "")
+      (reference "C7") (unit 1) (value "1 pF") (footprint "")
+    )
+    (path "/0e2270f1-03a5-4a80-b6d9-892401a77bc3"
+      (reference "C8") (unit 1) (value "22 pF") (footprint "")
     )
     (path "/00000000-0000-0000-0000-000061d0eeb6"
-      (reference "C7") (unit 1) (value "1 pF") (footprint "")
-    )
-    (path "/0e2270f1-03a5-4a80-b6d9-892401a77bc3"
-      (reference "C?") (unit 1) (value "22 pF") (footprint "")
+      (reference "C9") (unit 1) (value "1 pF") (footprint "")
     )
     (path "/00000000-0000-0000-0000-000061c95bc7"
