File: speech-synthesizer/schematics/speech-synthesizer/speech-synthesizer.kicad_sch (KiCad schematic)
At the start: 23 parts, among them Q1 2N4403, Q2 2N4403, U1 74LS245, U2 ATF22V10C, U3 74LS374, U4 74LS374, U5 TMS5220C

Commit message: working but noisy version
Parts:
- added U6: 74LS74, symbol 74xx:74LS74
Connections:
- net +5V: now also U6.10 (~{S}), U6.12 (D), U6.14 (VCC), U6.2 (D), U6.4 (~{S})
- net GND: now also U6.7 (GND); no longer U1.3 (A1), U1.6 (A4)
- net MODULE_BUSY: now also D3.2 (A)
- net RS: now also U1.6 (A4), U2.10 (IN9), U6.5 (Q); no longer U2.23 (I/O9), U5.28 (~{RS})
- net STATUSi: now also U2.18 (I/O4); no longer U2.19 (I/O5)
- net WS: now also U1.5 (A3), U2.11 (IN10), U6.9 (Q); no longer U2.22 (I/O8), U5.27 (~{WS})
- net ~{STATUSo}: now also U2.19 (I/O5); no longer U2.18 (I/O4)
- net ~{READY}: now reaches R3.2, U2.8 (IN7), U5.18 (~{READY})
- net ~{READY}: now also U1.3 (A1); no longer U1.4 (A2)
- net ~{INT}: now reaches R1.2, U2.9 (IN8), U5.17 (~{INT})
- net ~{INT}: now also U1.4 (A2); no longer U1.5 (A3)
- net DATAi renamed RS_RST
- net RS_RST: now also U6.1 (~{R}); no longer U4.11 (Cp)
- net ~{DATAa}: no longer names the net of U4.1 (OE)
- net ~{DATAa}: now also U5.27 (~{WS}), U6.8 (~{Q}); no longer U2.20 (I/O6)
- new net: U5.28 (~{RS}), U6.6 (~{Q})
- new net RS_CLK: U2.23 (I/O9), U6.3 (C)
- new net WS_CLK: U2.22 (I/O8), U4.11 (Cp), U6.11 (C)
- new net WS_RST: U2.20 (I/O6), U6.13 (~{R})
- no-connect marks 13 -> 12
Other:
- moved on the sheet: D3, R5
